File: hardware/KiCAD/KiCAD.kicad_sch (KiCad schematic)
At the start: 1 part, among them U1 STM32L021K4Tx

Commit message: update
Parts:
- added C1: 4u7, symbol Device:C_Small
- added C2, C3, C6: 100n, symbol Device:C_Small
- added C4: 1u, symbol Device:C_Small
- added C5: 10n, symbol Device:C_Small
- added D1: ~, symbol Device:LED_Small
- added L1: 39n, symbol Device:L_Small
- added R1: 1k, symbol Device:R_Small
- added R2: 100k, symbol Device:R_Small
Connections:
- net +3.3V: now also U1.17 (VDD), C1.1, C2.1, C3.1, L1.1
- net +3.3VA: now also C4.1, C5.1, L1.2
- net GND: now also C1.2, C2.2, C3.2, C4.2, C5.2, C6.2, R1.2, R2.2
- net NRST: now also C6.1
- net DAC_nCS: now reaches U1.10 (PA4)
- net SPI1_SCK: now reaches U1.11 (PA5)
- net SPI1_MOSI: now reaches U1.13 (PA7)
- net LED_STATUS: now reaches U1.18 (PA8)
- net LED_STATUS: now also D1.2 (A)
- net at U1.31 (PB9): now also R2.1
- net ADC_IN1: now reaches U1.7 (PA1)
- net DAC_nLDAC: now reaches U1.9 (PA3)
- new net: D1.1 (K), R1.1
Other:
- moved on the sheet: U1

Commit message: maj
Parts:
- added C10: 10u, symbol Device:C_Small
- added C7, C8: 1uF, symbol Device:C_Small
- added C9: 100n, symbol Device:C_Small
- added D2: GREEN LED, symbol Device:LED_Small
- added J1: Conn_02x07_Odd_Even, symbol Connector_Generic:Conn_02x07_Odd_Even
- added J2: POWER, symbol Connector_Generic:Conn_01x02
- added J3: INPUT, symbol Connector_Generic:Conn_01x02
- added J4: OUTPUT, symbol Connector_Generic:Conn_01x02
- added R3: 1k, symbol Device:R_Small
- added U2: BU33SD5WG-TR, Package_TO_SOT_SMD:SOT-23-5, symbol Regulator_Linear:MCP1802x-xx02xOT
- added U3: MCP4801-E/SN, symbol Analog_DAC:MCP4801
- D1: value ~ -> ORANGE
Connections:
- net +3.3V: now also C7.1, D2.2 (A), U2.5 (VOUT)
- net +3.3VA: now also C10.1, C9.1, U3.1 (Vdd), U3.6 (~{SHDN})
- net ADC_IN1: now also J3.1 (Pin_1)
- net DAC_nCS: now also U3.2 (~{CS})
- net DAC_nLDAC: now also U3.5 (~{LDAC})
- net GND: now also C10.2, C7.2, C8.2, C9.2, J1.11 (Pin_11), J1.5 (Pin_5), J1.7 (Pin_7), J2.2 (Pin_2), J3.2 (Pin_2), J4.2 (Pin_2), R3.2, U2.2 (GND), U3.7 (Vss)
- net NRST: now also J1.12 (Pin_12)
- net SPI1_MOSI: now also U3.4 (SDI)
- net SPI1_SCK: now also U3.3 (SCK)
- net SWDIO: now also J1.4 (Pin_4)
- net USART2_RX: now also J1.13 (Pin_13)
- net USART2_TX: now also J1.14 (Pin_14)
- new net: D2.1 (K), R3.1
- new net +5V: C8.1, J2.1 (Pin_1), U2.1 (VIN), U2.3 (~{SHDN})
- new net DAC_OUT: J4.1 (Pin_1), U3.8 (Vout)
- new net SWDCK: J1.6 (Pin_6)
- no-connect marks 0 -> 5
Other:
- moved on the sheet: C1, C2, C3, C4, C5, C6, D1, L1, R1, R2, U1
