File: hardware/KiCAD/KiCAD.kicad_sch (KiCad schematic)
At the start: 23 parts, among them J1 Conn_02x07_Odd_Even, J2 POWER, J3 INPUT, J4 OUTPUT, U1 STM32L021K4Tx, U2 BU33SD5WG-TR, U3 MCP4801-E/SN

Commit message: update
Parts:
- added H1, H2, H3, H4: MountingHole_Pad, MountingHole:MountingHole_3.2mm_M3_Pad, symbol Mechanical:MountingHole_Pad
- C1, C2, C3, C4, C5, C6, C9: footprint (none) -> Capacitor_SMD:C_0805_2012Metric_Pad1.18x1.45mm_HandSolder
- C10, C7, C8: footprint (none) -> Capacitor_SMD:C_0805_2012Metric
- D1, D2: footprint (none) -> LED_SMD:LED_0603_1608Metric_Pad1.05x0.95mm_HandSolder
- J1: footprint (none) -> Connector_PinHeader_1.27mm:PinHeader_2x07_P1.27mm_Vertical_SMD
- J2, J3, J4: footprint (none) -> Connector_JST:JST_XH_B2B-XH-A_1x02_P2.50mm_Vertical
- L1: footprint (none) -> Inductor_SMD:L_0805_2012Metric_Pad1.05x1.20mm_HandSolder
- R1, R2, R3: footprint (none) -> Resistor_SMD:R_0805_2012Metric_Pad1.20x1.40mm_HandSolder
- U3: footprint (none) -> Package_SO:SOIC-8_3.9x4.9mm_P1.27mm
Connections:
- net +3.3V: now also J1.3 (Pin_3)
- net GND: now also H1.1, H2.1, H3.1, H4.1
- no-connect marks 5 -> 20
