File: hardware/KiCAD/KiCAD.kicad_sch (KiCad schematic)
At the start: 27 parts, among them J1 Conn_02x07_Odd_Even, J2 POWER, J3 INPUT, J4 OUTPUT, U1 STM32L021K4Tx, U2 BU33SD5WG-TR, U3 MCP4801-E/SN

Commit message: update2
Parts:
- C10, C7, C8: footprint Capacitor_SMD:C_0805_2012Metric -> Capacitor_SMD:C_0805_2012Metric_Pad1.18x1.45mm_HandSolder
- R1: value 1k -> 180
Connections:
- net SWDCK is gone; now on net SWCLK: J1.6 (Pin_6)
Other:
- note added: "Placez les 100n au plus proche du pin"
Changed lines of the file:
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@@
   )
   (rectangle (start 204.47 13.97) (end 283.21 62.23)
-    (stroke (width 0) (type default))
+    (stroke (width 0) (type dot))
     (fill (type none))
+  )
+  (text "Placez les 100n au plus proche du pin " (at 26.67 33.02 0)
+    (effects (font (size 1.27 1.27)) (justify left bottom))
   )
   (text "Connectors\n" (at 205.74 74.93 0)
@@
     )
   )
-  (global_label "SWDCK" (shape input) (at 157.48 113.03 0) (fields_autoplaced)
-    (effects (font (size 1.27 1.27)) (justify left))
-    (property "Intersheetrefs" "${INTERSHEET_REFS}" (at 166.9361 113.03 0)
+  (global_label "SWCLK" (shape input) (at 157.48 113.03 0) (fields_autoplaced)
+    (effects (font (size 1.27 1.27)) (justify left))
+    (property "Intersheetrefs" "${INTERSHEET_REFS}" (at 166.6942 113.03 0)
       (effects (font (size 1.27 1.27)) (justify left) hide)
     )
@@
       (effects (font (size 1.27 1.27)) (justify left))
     )
-    (property "Footprint" "Capacitor_SMD:C_0805_2012Metric" (at 213.36 29.21 0)
+    (property "Footprint" "Capacitor_SMD:C_0805_2012Metric_Pad1.18x1.45mm_HandSolder" (at 213.36 29.21 0)
       (effects (font (size 1.27 1.27)) hide)
     )
@@
       (effects (font (size 1.27 1.27)) (justify left))
     )
-    (property "Value" "1k" (at 35.56 92.71 0)
+    (property "Value" "180" (at 35.56 92.71 0)
       (effects (font (size 1.27 1.27)) (justify left))
     )
@@
       (effects (font (size 1.27 1.27)) (justify left))
     )
-    (property "Footprint" "Capacitor_SMD:C_0805_2012Metric" (at 247.65 30.48 0)
+    (property "Footprint" "Capacitor_SMD:C_0805_2012Metric_Pad1.18x1.45mm_HandSolder" (at 247.65 30.48 0)
       (effects (font (size 1.27 1.27)) hide)
     )
@@
       (effects (font (size 1.27 1.27)) (justify left))
     )
-    (property "Footprint" "Capacitor_SMD:C_0805_2012Metric" (at 186.69 26.67 0)
-      (effects (font (size 1.27 1.27)) hide)
-    )
+    (property "Footprint" "Capacitor_SMD:C_0805_2012Metric_Pad1.18x1.45mm_HandSolder" (at 186.69 26.67 0)
+      (effects (font (size 1.27 1.27)) hide)
+    )

Commit message: update3
Other:
- moved on the sheet: C8
Changed lines of the file:
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@@
   (junction (at 97.79 22.86) (diameter 0) (color 0 0 0 0)
   )
-  (junction (at 213.36 24.13) (diameter 0) (color 0 0 0 0)
+  (junction (at 209.55 24.13) (diameter 0) (color 0 0 0 0)
   )
   (junction (at 85.09 22.86) (diameter 0) (color 0 0 0 0)
@@
   (junction (at 68.58 44.45) (diameter 0) (color 0 0 0 0)
   )
-  (junction (at 213.36 38.1) (diameter 0) (color 0 0 0 0)
+  (junction (at 209.55 38.1) (diameter 0) (color 0 0 0 0)
   )
   (junction (at 63.5 152.4) (diameter 0) (color 0 0 0 0)
@@
   (junction (at 148.59 41.91) (diameter 0) (color 0 0 0 0)
   )
+  (junction (at 217.17 24.13) (diameter 0) (color 0 0 0 0)
+  )
   (junction (at 247.65 24.13) (diameter 0) (color 0 0 0 0)
   )
@@
   )
   (junction (at 231.14 38.1) (diameter 0) (color 0 0 0 0)
+  )
+  (junction (at 217.17 38.1) (diameter 0) (color 0 0 0 0)
   )
   (junction (at 21.59 22.86) (diameter 0) (color 0 0 0 0)
@@
     (stroke (width 0) (type default))
   )
-  (wire (pts (xy 213.36 38.1) (xy 231.14 38.1))
+  (wire (pts (xy 209.55 38.1) (xy 217.17 38.1))
     (stroke (width 0) (type default))
   )
@@
     (stroke (width 0) (type default))
   )
-  (wire (pts (xy 213.36 24.13) (xy 213.36 26.67))
+  (wire (pts (xy 209.55 24.13) (xy 209.55 26.67))
     (stroke (width 0) (type default))
   )
@@
     (stroke (width 0) (type default))
   )
-  (wire (pts (xy 213.36 31.75) (xy 213.36 38.1))
+  (wire (pts (xy 209.55 31.75) (xy 209.55 38.1))
     (stroke (width 0) (type default))
   )
@@
     (stroke (width 0) (type default))
   )
-  (wire (pts (xy 213.36 24.13) (xy 220.98 24.13))
+  (wire (pts (xy 209.55 24.13) (xy 217.17 24.13))
     (stroke (width 0) (type default))
   )
@@
     (stroke (width 0) (type default))
   )
+  (wire (pts (xy 217.17 38.1) (xy 231.14 38.1))
+    (stroke (width 0) (type default))
+  )
   (wire (pts (xy 63.5 143.51) (xy 63.5 152.4))
     (stroke (width 0) (type default))
@@
   )
   (wire (pts (xy 237.49 90.17) (xy 241.3 90.17))
+    (stroke (width 0) (type default))
+  )
+  (wire (pts (xy 217.17 24.13) (xy 220.98 24.13))
     (stroke (width 0) (type default))
   )
@@
     )
   )
-  (symbol (lib_id "power:GND") (at 213.36 38.1 0) (unit 1)
-    (in_bom yes) (on_board yes) (dnp no) (fields_autoplaced)
-    (property "Reference" "#PWR013" (at 213.36 44.45 0)
-      (effects (font (size 1.27 1.27)) hide)
-    )
-    (property "Value" "GND" (at 213.36 43.18 0)
-      (effects (font (size 1.27 1.27)))
-    )
-    (property "Footprint" "" (at 213.36 38.1 0)
-      (effects (font (size 1.27 1.27)) hide)
-    )
-    (property "Datasheet" "" (at 213.36 38.1 0)
+  (symbol (lib_id "power:GND") (at 209.55 38.1 0) (unit 1)
+    (in_bom yes) (on_board yes) (dnp no) (fields_autoplaced)
+    (property "Reference" "#PWR013" (at 209.55 44.45 0)
+      (effects (font (size 1.27 1.27)) hide)
+    )
+    (property "Value" "GND" (at 209.55 43.18 0)
+      (effects (font (size 1.27 1.27)))
+    )
+    (property "Footprint" "" (at 209.55 38.1 0)
+      (effects (font (size 1.27 1.27)) hide)
+    )
+    (property "Datasheet" "" (at 209.55 38.1 0)
       (effects (font (size 1.27 1.27)) hide)
     )
@@
     )
   )
-  (symbol (lib_id "Device:C_Small") (at 213.36 29.21 0) (unit 1)
-    (in_bom yes) (on_board yes) (dnp no) (fields_autoplaced)
-    (property "Reference" "C8" (at 215.9 27.9463 0)
-      (effects (font (size 1.27 1.27)) (justify left))
-    )
-    (property "Value" "1uF" (at 215.9 30.4863 0)
-      (effects (font (size 1.27 1.27)) (justify left))
-    )
-    (property "Footprint" "Capacitor_SMD:C_0805_2012Metric_Pad1.18x1.45mm_HandSolder" (at 213.36 29.21 0)
-      (effects (font (size 1.27 1.27)) hide)
-    )
-    (property "Datasheet" "~" (at 213.36 29.21 0)
+  (symbol (lib_id "Device:C_Small") (at 209.55 29.21 0) (unit 1)
+    (in_bom yes) (on_board yes) (dnp no) (fields_autoplaced)
+    (property "Reference" "C8" (at 212.09 27.9463 0)
+      (effects (font (size 1.27 1.27)) (justify left))
+    )
+    (property "Value" "1uF" (at 212.09 30.4863 0)
+      (effects (font (size 1.27 1.27)) (justify left))
+    )
+    (property "Footprint" "Capacitor_SMD:C_0805_2012Metric_Pad1.18x1.45mm_HandSolder" (at 209.55 29.21 0)
+      (effects (font (size 1.27 1.27)) hide)
+    )
+    (property "Datasheet" "~" (at 209.55 29.21 0)
       (effects (font (size 1.27 1.27)) hide)
     )
@@
     )
   )
-  (symbol (lib_id "power:+5V") (at 213.36 24.13 0) (unit 1)
-    (in_bom yes) (on_board yes) (dnp no) (fields_autoplaced)
-    (property "Reference" "#PWR012" (at 213.36 27.94 0)
-      (effects (font (size 1.27 1.27)) hide)
-    )
-    (property "Value" "+5V" (at 213.36 19.05 0)
-      (effects (font (size 1.27 1.27)))
-    )
-    (property "Footprint" "" (at 213.36 24.13 0)
-      (effects (font (size 1.27 1.27)) hide)
-    )
-    (property "Datasheet" "" (at 213.36 24.13 0)
+  (symbol (lib_id "power:+5V") (at 209.55 24.13 0) (unit 1)
+    (in_bom yes) (on_board yes) (dnp no) (fields_autoplaced)
+    (property "Reference" "#PWR012" (at 209.55 27.94 0)
+      (effects (font (size 1.27 1.27)) hide)
+    )
+    (property "Value" "+5V" (at 209.55 19.05 0)
+      (effects (font (size 1.27 1.27)))
+    )
+    (property "Footprint" "" (at 209.55 24.13 0)
+      (effects (font (size 1.27 1.27)) hide)
+    )
+    (property "Datasheet" "" (at 209.55 24.13 0)
       (effects (font (size 1.27 1.27)) hide)
     )
@@
         (path "/f237dfd5-d4df-457f-ad80-4bb95ef52d08"
           (reference "C1") (unit 1)
+        )
+      )
+    )
+  )
+  (symbol (lib_id "power:PWR_FLAG") (at 85.09 22.86 0) (unit 1)
+    (in_bom yes) (on_board yes) (dnp no) (fields_autoplaced)
+    (property "Reference" "#FLG01" (at 85.09 20.955 0)
+      (effects (font (size 1.27 1.27)) hide)
+    )
+    (property "Value" "PWR_FLAG" (at 85.09 17.78 0)
+      (effects (font (size 1.27 1.27)))
+    )
+    (property "Footprint" "" (at 85.09 22.86 0)
+      (effects (font (size 1.27 1.27)) hide)
+    )
+    (property "Datasheet" "~" (at 85.09 22.86 0)
+      (effects (font (size 1.27 1.27)) hide)
+    )
+    (pin "1")
+    (instances
+      (project "KiCAD"
+        (path "/f237dfd5-d4df-457f-ad80-4bb95ef52d08"
+          (reference "#FLG01") (unit 1)
         )
       )
@@
     )
   )
+  (symbol (lib_id "power:PWR_FLAG") (at 217.17 24.13 0) (unit 1)
+    (in_bom yes) (on_board yes) (dnp no) (fields_autoplaced)
+    (property "Reference" "#FLG02" (at 217.17 22.225 0)
+      (effects (font (size 1.27 1.27)) hide)
+    )
+    (property "Value" "PWR_FLAG" (at 217.17 19.05 0)
+      (effects (font (size 1.27 1.27)))
+    )
+    (property "Footprint" "" (at 217.17 24.13 0)
+      (effects (font (size 1.27 1.27)) hide)
+    )
+    (property "Datasheet" "~" (at 217.17 24.13 0)
+      (effects (font (size 1.27 1.27)) hide)
+    )
+    (pin "1")
+    (instances
+      (project "KiCAD"
+        (path "/f237dfd5-d4df-457f-ad80-4bb95ef52d08"
+          (reference "#FLG02") (unit 1)
+        )
+      )
+    )
+  )
   (symbol (lib_id "power:GND") (at 148.59 67.31 0) (unit 1)
     (in_bom yes) (on_board yes) (dnp no) (fields_autoplaced)
@@
         )
       )
+    )
+  )
+  (symbol (lib_id "power:PWR_FLAG") (at 217.17 38.1 180) (unit 1)
+    (in_bom yes) (on_board yes) (dnp no) (fields_autoplaced)
+    (property "Reference" "#FLG03" (at 217.17 40.005 0)
+      (effects (font (size 1.27 1.27)) hide)
+    )
+    (property "Value" "PWR_FLAG" (at 217.17 43.18 0)
+      (effects (font (size 1.27 1.27)))
+    )
+    (property "Footprint" "" (at 217.17 38.1 0)
+      (effects (font (size 1.27 1.27)) hide)
+    )
+    (property "Datasheet" "~" (at 217.17 38.1 0)
+      (effects (font (size 1.27 1.27)) hide)
+    )
+    (pin "1")
+    (instances
+      (project "KiCAD"
+        (path "/f237dfd5-d4df-457f-ad80-4bb95ef52d08"
+          (reference "#FLG03") (unit 1)
+        )
+      )
