File: hardware/KiCAD/KiCAD.kicad_pcb (KiCad board)
At the start: 2 copper layers, 27 parts, among them J1 Conn_02x07_Odd_Even, J2 POWER, J3 INPUT, J4 OUTPUT, U1 STM32L021K4Tx, U2 BU33SD5WG-TR, U3 MCP4801-E/SN

Commit message: update
Parts:
- C1: value 4u7 -> 10u
- C5: value 10n -> 100n
- R1: value 1k -> 180
- R3: value 1k -> 240
- moved U2 97.4 mm to (95.1, 45.0)
- moved C8 93.2 mm to (94.0, 49.0), turned to -90 degrees
- moved C7 89.5 mm to (99.0, 44.0)
- moved C10 82.4 mm to (99.0, 71.0), turned to -90 degrees
- moved R1 79.7 mm to (93.0, 59.0), turned to -90 degrees
- moved U3 77.7 mm to (109.6, 49.5), turned to -90 degrees
- moved R2 76.1 mm to (103.0, 52.0), turned to 90 degrees
- moved C9 72.0 mm to (96.0, 70.0), turned to 180 degrees
- moved D1 70.2 mm to (95.9, 58.0)
- moved L1 69.9 mm to (98.0, 63.1), turned to -90 degrees
- moved C1 69.0 mm to (98.3, 54.5), turned to 90 degrees
- moved C3 68.8 mm to (100.4, 54.5), turned to 90 degrees
- moved J1 63.5 mm to (121.0, 50.0), turned to 90 degrees
- moved C5 57.8 mm to (113.0, 59.0)
- moved R3 57.4 mm to (118.0, 66.0)
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Routing:
- net GND: vias 0 -> 1
- added copper zone on B.Cu, net GND
- added copper zone on F.Cu, net GND
Other:
- board outline added: 58 x 48 mm
