File: hardware/KiCAD/KiCAD.kicad_pcb (KiCad board)
At the start: 2 copper layers, 58 x 48 mm, 27 parts, among them J1 Conn_02x07_Odd_Even, J2 POWER, J3 INPUT, J4 OUTPUT, U1 STM32L021K4Tx, U2 BU33SD5WG-TR, U3 MCP4801-E/SN

Commit message: update3
Parts:
- moved J1 40.7 mm to (90.6, 72.5)
- moved R1 5.15 mm to (112.3, 59.9), turned to 180 degrees
- moved C6 2.25 mm to (97.1, 59.7), turned to 90 degrees
- moved D1 0.65 mm to (112.3, 61.7)
Connections:
- J1 pad 6: SWDCK -> SWCLK
Routing:
- net SWDIO: track 0.00 -> 36.3 mm, vias 0 -> 2
- net SWCLK: track 0.00 -> 30.5 mm, vias 0 -> 2
- net ADC_IN1: track 0.00 -> 28.7 mm
- net NRST: track 0.00 -> 24.8 mm, vias 0 -> 2
- net USART2_RX: track 0.00 -> 21.9 mm, vias 0 -> 2
- net +3.3V: track 56.1 -> 74.9 mm, vias 0 -> 2
- net USART2_TX: track 0.00 -> 11.6 mm
- net GND: track 0.00 -> 2.48 mm, vias 0 -> 1
- net LED_STATUS: track 0.00 -> 2.25 mm
- net Net-(D1-K): track 0.00 -> 1.85 mm
- net +3.3VA: track 32.8 -> 33.9 mm, vias 0 -> 2
