File: hardware/KiCAD/_autosave-KiCAD.kicad_sch (KiCad schematic)
At the start: 27 parts, among them J1 Conn_02x07_Odd_Even, J2 POWER, J3 INPUT, J4 OUTPUT, U1 STM32L021K4Tx, U2 BU33SD5WG-TR, U3 MCP4801-E/SN

Commit message: update
Parts:
- R1: value 1k -> 180
Other:
- note added: "Placez les 100n au plus proche du pin"
Changed lines of the file:
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@@
   )
   (rectangle (start 204.47 13.97) (end 283.21 62.23)
-    (stroke (width 0) (type default))
+    (stroke (width 0) (type dot))
     (fill (type none))
+  )
+  (text "Placez les 100n au plus proche du pin " (at 26.67 33.02 0)
+    (effects (font (size 1.27 1.27)) (justify left bottom))
   )
   (text "Connectors\n" (at 205.74 74.93 0)
@@
       (effects (font (size 1.27 1.27)) (justify left))
     )
-    (property "Value" "1k" (at 35.56 92.71 0)
-      (effects (font (size 1.27 1.27)) (justify left))
-    )
+    (property "Value" "180" (at 35.56 92.71 0)
+      (effects (font (size 1.27 1.27)) (justify left))
+    )
